Commit message: base test imu and lidar success

File: src/robot_description/urdf/agv_base.urdf (robot description, URDF)
Before this commit: robot robot, 6 links, 5 joints
Links:
- link left_wheel_link: geometry visual cylinder length=0.04 radius=0.105
- link right_wheel_link: geometry visual cylinder length=0.04 radius=0.105
Joints:
- joint caster_joint: child front_caster_link -> caster_link; origin xyz=0.37 0 0 rpy=0 0 0 -> xyz=0.33 0 0 rpy=0 0 0
- joint laser_joint: origin xyz=0 0 0.15 rpy=0 0 0 -> xyz=0 0 0.15 rpy=0 0 3.1415926
- joint left_wheel_joint: origin xyz=-0.185 0 0 rpy=0 0 0 -> xyz=0 0.1825 0 rpy=0 0 0
- joint right_wheel_joint: origin xyz=0.185 0 0 rpy=0 0 0 -> xyz=0 -0.1825 0 rpy=0 0 0

Commit message: nav_V1

File: src/robot_description/urdf/agv_base.urdf (robot description, URDF)
Before this commit: robot robot, 6 links, 5 joints
Joints:
- joint laser_joint: origin xyz=0 0 0.15 rpy=0 0 3.1415926 -> xyz=0 0 0.15 rpy=0 3.1415926 0

Commit message: 10.25

File: src/robot_description/urdf/agv_base.urdf (robot description, URDF)
Before this commit: robot robot, 6 links, 5 joints
Links:
- added link camera_link; visual box size=0.02 0.15 0.02
Joints:
- added joint camera_joint: type fixed, parent base_link, child camera_link, origin xyz=0.45 0.05 0.1 rpy=0 0 0

Commit message: 1028

File: src/robot_description/urdf/agv_base.urdf (robot description, URDF)
Before this commit: robot robot, 7 links, 6 joints
Joints:
- joint camera_joint: origin xyz=0.45 0.05 0.1 rpy=0 0 0 -> xyz=0.45 0.06 0.1 rpy=0 0 0

Commit message: 11/5

File: src/robot_description/urdf/agv_base.urdf (robot description, URDF)
Before this commit: robot robot, 7 links, 6 joints
Joints:
- joint imu_joint: origin xyz=0 0 0 -> xyz=0 0 0 rpy=0 0 0
