Commit message: 02/25/gazebo

File: src/urdf_agv_description/urdf/agv_base_gazebo.urdf (robot description, URDF)
Before this commit: robot robot, 6 links, 5 joints
Links:
- added link base_footprint
Joints:
- added joint base_joint: type fixed, parent base_footprint, child base_link, origin xyz=0.0 0.0 0.07 rpy=0 0 0

Commit message: 0307_2

File: src/urdf_agv_description/urdf/agv_base_gazebo.urdf (robot description, URDF)
Before this commit: robot robot, 6 links, 5 joints
Links:
- link base_link: mass 0.2 -> 0.8
- link caster_link: mass 0.02 -> 0.5
- link imu_link: mass 0.1 -> 0.01
