Commit message: 0307

File: src/urdf_agv_description/urdf/agv_base.urdf (robot description, URDF)
Before this commit: robot robot, 7 links, 6 joints
Joints:
- joint laser_joint: axis (none) -> 0 0 1; type fixed -> continuous
- joint left_wheel_joint: origin xyz=0 0.1825 0 rpy=0 0 0 -> xyz=0 0.179 0 rpy=0 0 0
- joint right_wheel_joint: origin xyz=0 -0.1825 0 rpy=0 0 0 -> xyz=0 -0.179 0 rpy=0 0 0

File: src/urdf_agv_description/urdf/agv_base_gazebo.urdf (robot description, URDF)
Before this commit: robot robot, 6 links, 5 joints
Joints:
- joint laser_joint: origin xyz=0 0 0.15 rpy=0 3.1415926 0 -> xyz=0 0 0.15 rpy=0 0 0

Commit message: 03/12

File: src/urdf_agv_description/urdf/agv_base.urdf (robot description, URDF)
Before this commit: robot robot, 7 links, 6 joints
Joints:
- joint laser_joint: axis 0 0 1 -> (none); type continuous -> fixed
